File: Black_STM32F407VET6/STM32F407VET6.sch (KiCad schematic (older format))
At the start: 102 parts, among them J1 T0, J10 Fan2, J11 Fan1, J12 X_logic, J13 Microsteps, J14 X-, J15 Y-, J16 Z-, J17 Left, J18 Y_logic, J19 X+, J2 T1, J20 Y+, J21 Z+, J22 Microsteps, J23 EXP2, J24 Z_logic, J25 Bottom, J26 Microsteps, J27 EXP1, J28 E0_logic, J29 Microsteps, J3 TB, J30 Right, J31 E1_logic, J32 Microsteps, J33 X_motor, J34 Y_motor, J35 Z_motor, J36 E0_motor, J37 E1_motor, J38 X, J39 Y, J4 TC, J40 Z, J41 E0, J42 E1, J43 Fan0, J44 COM, J45 USB, J47 I2C, J48 SPI, J49 SPI, J5 + VIN -, J50 SDIO, J51 Servo, J52 Servo, J53 PowerSelect, J54 Power, J55 PD11, J56 Power, J6 - HotBed +, J7 Heater0, J8 Heater1, J9 Fan3, Q1 IRLR8726PBF, Q2 IRLR8726PBF, Q3 IRLR8726PBF, Q4 IRLML0030TRPBF, Q5 IRLML0030TRPBF, Q6 IRLML0030TRPBF, Q7 IRLML0030TRPBF, U1 SN74AHC, U2 SN74AHC, U3 SN74AHC, U4 LM2596S-5, U5 AT24CS01-SSHM

Commit message: change dcdc chip
Parts:
- removed C5: 100uF 35V, Capacitor_THT:CP_Radial_D8.0mm_P3.50mm, symbol Device:CP_Small
- removed C6: 220uF 35V, Capacitor_THT:CP_Radial_D6.3mm_P2.50mm, symbol Device:CP_Small
- removed D1: SS14, Diode_SMD:D_SMA, symbol Diode:B120-E3
- removed L1: 47uH, Inductor_THT:L_Radial_D9.5mm_P5.00mm_Fastron_07HVP, symbol Device:L_Small
- removed U4: LM2596S-5, Package_TO_SOT_SMD:TO-263-5_TabPin3, symbol Regulator_Switching:LM2596S-5
- C1, C2, C3, C4: footprint Capacitor_THT:CP_Radial_D5.0mm_P2.00mm -> Capacitor_Tantalum_SMD:CP_EIA-3216-10_Kemet-I
Connections:
- wire segments 180 -> 171
Other:
- moved on the sheet: J5, J8
Changed lines of the file:
@@
 EESchema Schematic File Version 4
-EELAYER 26 0
+LIBS:STM32F407VET6-cache
+EELAYER 29 0
 EELAYER END
 $Descr A4 11693 8268
 encoding utf-8
-Sheet 1 1
+Sheet 1 2
 Title ""
 Date ""
@@
 L Connector:Screw_Terminal_01x02 J8
 U 1 1 5C4B2565
-P 2300 5200
-F 0 "J8" H 2380 5192 50  0000 L CNN
-F 1 "Heater1" H 2380 5101 50  0000 L CNN
-F 2 "TerminalBlock_MetzConnect:TerminalBlock_MetzConnect_Type059_RT06302HBWC_1x02_P3.50mm_Horizontal" H 2300 5200 50  0001 C CNN
-F 3 "~" H 2300 5200 50  0001 C CNN
-	1    2300 5200
+P 2450 5150
+F 0 "J8" H 2530 5142 50  0000 L CNN
+F 1 "Heater1" H 2530 5051 50  0000 L CNN
+F 2 "TerminalBlock_MetzConnect:TerminalBlock_MetzConnect_Type059_RT06302HBWC_1x02_P3.50mm_Horizontal" H 2450 5150 50  0001 C CNN
+F 3 "~" H 2450 5150 50  0001 C CNN
+	1    2450 5150
 	1    0    0    -1
 $EndComp
@@
 L Connector:Screw_Terminal_01x02 J5
 U 1 1 5C4B4AC4
-P 2300 3850
-F 0 "J5" H 2380 3842 50  0000 L CNN
-F 1 "+ VIN -" H 2380 3751 50  0000 L CNN
-F 2 "TerminalBlock_MetzConnect:TerminalBlock_MetzConnect_Type055_RT01502HDWU_1x02_P5.00mm_Horizontal" H 2300 3850 50  0001 C CNN
-F 3 "~" H 2300 3850 50  0001 C CNN
-	1    2300 3850
+P 2300 3800
+F 0 "J5" H 2380 3792 50  0000 L CNN
+F 1 "+ VIN -" H 2380 3701 50  0000 L CNN
+F 2 "TerminalBlock_MetzConnect:TerminalBlock_MetzConnect_Type055_RT01502HDWU_1x02_P5.00mm_Horizontal" H 2300 3800 50  0001 C CNN
+F 3 "~" H 2300 3800 50  0001 C CNN
+	1    2300 3800
 	1    0    0    -1
 $EndComp
@@
 $EndComp
 Wire Wire Line
-	1900 4100 2100 4100
-Wire Wire Line
-	1900 4650 2100 4650
-Wire Wire Line
-	1900 5200 2100 5200
-Wire Wire Line
-	2100 5300 2050 5300
-Wire Wire Line
-	2050 5300 2050 4750
-Wire Wire Line
-	2050 3950 2100 3950
-Wire Wire Line
-	2100 4200 2050 4200
-Connection ~ 2050 4200
-Wire Wire Line
-	2050 4200 2050 3950
+	2250 5250 2050 5250
+Wire Wire Line
+	2050 5250 2050 4750
+Wire Wire Line
+	2050 3900 2100 3900
 Wire Wire Line
 	2100 4750 2050 4750
 Connection ~ 2050 4750
 Wire Wire Line
-	2050 4750 2050 4200
-Wire Wire Line
-	2000 3850 2100 3850
+	2000 3800 2100 3800
 Wire Wire Line
 	1900 5050 2000 5050
-Wire Wire Line
-	2000 5050 2000 4500
-Wire Wire Line
-	1900 4450 1900 4500
-Wire Wire Line
-	1900 4500 2000 4500
-Connection ~ 2000 4500
-Wire Wire Line
-	2000 4500 2000 3850
 $Comp
 L Device:Q_NMOS_GSD Q4
@@
 F 0 "C1" H 1300 6100 50  0000 L CNN
 F 1 "10uF 16V" H 1300 6200 50  0000 L CNN
-F 2 "Capacitor_THT:CP_Radial_D5.0mm_P2.00mm" H 1200 6150 50  0001 C CNN
+F 2 "Capacitor_Tantalum_SMD:CP_EIA-3216-10_Kemet-I" H 1200 6150 50  0001 C CNN
 F 3 "~" H 1200 6150 50  0001 C CNN
 	1    1200 6150
@@
 F 0 "C2" H 1112 6554 50  0000 R CNN
 F 1 "10uF 16V" H 1112 6645 50  0000 R CNN
-F 2 "Capacitor_THT:CP_Radial_D5.0mm_P2.00mm" H 1200 6600 50  0001 C CNN
+F 2 "Capacitor_Tantalum_SMD:CP_EIA-3216-10_Kemet-I" H 1200 6600 50  0001 C CNN
 F 3 "~" H 1200 6600 50  0001 C CNN
 	1    1200 6600
@@
 F 0 "C3" H 1112 7004 50  0000 R CNN
 F 1 "10uF 16V" H 1112 7095 50  0000 R CNN
-F 2 "Capacitor_THT:CP_Radial_D5.0mm_P2.00mm" H 1200 7050 50  0001 C CNN
+F 2 "Capacitor_Tantalum_SMD:CP_EIA-3216-10_Kemet-I" H 1200 7050 50  0001 C CNN
 F 3 "~" H 1200 7050 50  0001 C CNN
 	1    1200 7050
@@
 F 0 "C4" H 1112 7454 50  0000 R CNN
 F 1 "10uF 16V" H 1112 7545 50  0000 R CNN
-F 2 "Capacitor_THT:CP_Radial_D5.0mm_P2.00mm" H 1200 7500 50  0001 C CNN
+F 2 "Capacitor_Tantalum_SMD:CP_EIA-3216-10_Kemet-I" H 1200 7500 50  0001 C CNN
 F 3 "~" H 1200 7500 50  0001 C CNN
 	1    1200 7500
 	-1   0    0    -1
-$EndComp
-$Comp
-L Regulator_Switching:LM2596S-5 U4
-U 1 1 5C508FEC
-P 7450 5800
-F 0 "U4" H 7450 6167 50  0000 C CNN
-F 1 "LM2596S-5" H 7450 6076 50  0000 C CNN
-F 2 "Package_TO_SOT_SMD:TO-263-5_TabPin3" H 7500 5550 50  0001 L CIN
-F 3 "http://www.ti.com/lit/ds/symlink/lm2596.pdf" H 7450 5800 50  0001 C CNN
-	1    7450 5800
-	1    0    0    -1
-$EndComp
-$Comp
-L Device:CP_Small C5
-U 1 1 5C50912F
-P 6750 6050
-F 0 "C5" H 6838 6096 50  0000 L CNN
-F 1 "100uF 35V" H 6838 6005 50  0000 L CNN
-F 2 "Capacitor_THT:CP_Radial_D8.0mm_P3.50mm" H 6750 6050 50  0001 C CNN
-F 3 "~" H 6750 6050 50  0001 C CNN
-	1    6750 6050
-	-1   0    0    -1
-$EndComp
-$Comp
-L Device:CP_Small C6
-U 1 1 5C509233
-P 8450 6050
-F 0 "C6" H 8538 6096 50  0000 L CNN
-F 1 "220uF 35V" H 8538 6005 50  0000 L CNN
-F 2 "Capacitor_THT:CP_Radial_D6.3mm_P2.50mm" H 8450 6050 50  0001 C CNN
-F 3 "~" H 8450 6050 50  0001 C CNN
-	1    8450 6050
-	1    0    0    -1
-$EndComp
-$Comp
-L Device:L_Small L1
-U 1 1 5C50C0B1
-P 8250 5900
-F 0 "L1" H 8297 5946 50  0000 L CNN
-F 1 "47uH" H 8297 5855 50  0000 L CNN
-F 2 "Inductor_THT:L_Radial_D9.5mm_P5.00mm_Fastron_07HVP" H 8250 5900 50  0001 C CNN
-F 3 "~" H 8250 5900 50  0001 C CNN
-	1    8250 5900
-	0    -1   -1   0
 $EndComp
 Wire Wire Line
@@
 	1500 5400 1600 5400
 Wire Wire Line
-	8450 6200 8450 6150
-$Comp
-L Diode:B120-E3 D1
-U 1 1 5C51EDB0
-P 8050 6050
-F 0 "D1" V 8004 6129 50  0000 L CNN
-F 1 "SS14" V 8095 6129 50  0000 L CNN
-F 2 "Diode_SMD:D_SMA" H 8050 5875 50  0001 C CNN
-F 3 "http://www.vishay.com/docs/88946/b120.pdf" H 8050 6050 50  0001 C CNN
-	1    8050 6050
-	0    1    1    0
-$EndComp
-Wire Wire Line
-	8450 6200 8050 6200
-Wire Wire Line
-	7450 6200 7450 6100
-Connection ~ 8050 6200
-Wire Wire Line
-	8050 6200 7450 6200
-Wire Wire Line
-	7450 6200 6950 6200
-Wire Wire Line
-	6750 6200 6750 6150
-Connection ~ 7450 6200
-Wire Wire Line
-	6950 5900 6950 6200
-Connection ~ 6950 6200
-Wire Wire Line
-	6950 6200 6750 6200
-Wire Wire Line
-	6750 5950 6750 5700
-Wire Wire Line
-	6750 5700 6950 5700
-Wire Wire Line
-	7950 5900 8050 5900
-Connection ~ 8050 5900
-Wire Wire Line
-	8050 5900 8150 5900
-Wire Wire Line
-	7950 5700 8450 5700
-Wire Wire Line
-	8450 5700 8450 5900
-Wire Wire Line
-	8350 5900 8450 5900
-Connection ~ 8450 5900
-Wire Wire Line
-	8450 5900 8450 5950
-Wire Wire Line
 	4100 1100 4100 1200
 Wire Wire Line
@@
 Text GLabel 900  5400 0    50   Input ~ 0
 GND
-Text GLabel 2050 3750 1    50   Input ~ 0
+Text GLabel 2050 3500 1    50   Input ~ 0
 12V
 Wire Wire Line
-	2050 3750 2050 3950
-Connection ~ 2050 3950
-Text GLabel 2000 3850 0    50   Input ~ 0
+	2050 3500 2050 3900
+Connection ~ 2050 3900
+Text GLabel 1900 3800 0    50   Input ~ 0
 GND
 Text GLabel 5600 3550 1    50   Input ~ 0
@@
 Text GLabel 3650 5850 1    50   Input ~ 0
 GND
-Text GLabel 6750 5700 1    50   Input ~ 0
-12V
-Text GLabel 8450 5700 1    50   Input ~ 0
-5V
 Wire Wire Line
 	1150 2250 1250 2250
@@
 	7350 800  7350 1100
 Connection ~ 7100 800
-Text GLabel 7450 6200 3    50   Input ~ 0
-GND
 $Comp
 L Device:Q_NMOS_GSD Q7
@@
 U 1 1 5C614ADE
 P 10650 1750
-F 0 "R18" H 10591 1704 50  0000 R CNN
-F 1 "22R" H 10591 1795 50  0000 R CNN
+F 0 "R18" H 10850 2100 50  0000 R CNN
+F 1 "22R" H 10850 2000 50  0000 R CNN
 F 2 "Resistor_SMD:R_0603_1608Metric" H 10650 1750 50  0001 C CNN
 F 3 "~" H 10650 1750 50  0001 C CNN
@@
 U 1 1 5C61CFBD
 P 10650 1850
-F 0 "R19" H 10591 1804 50  0000 R CNN
-F 1 "22R" H 10591 1895 50  0000 R CNN
+F 0 "R19" H 10600 2200 50  0000 R CNN
+F 1 "22R" H 10600 2100 50  0000 R CNN
 F 2 "Resistor_SMD:R_0603_1608Metric" H 10650 1850 50  0001 C CNN
 F 3 "~" H 10650 1850 50  0001 C CNN
@@
 Connection ~ 850  2050
 Connection ~ 850  2600
-Connection ~ 1900 4500
 Connection ~ 1250 2250
 Connection ~ 1300 1750
@@
 	1300 2300 1300 3100
 Connection ~ 1300 2300
+$Sheet
+S 7100 5150 550  500
+U 5D345ACA
+F0 "POWER" 50
+F1 "power.sch" 50
+F2 "12V" I L 7100 5400 50
+F3 "5V" O R 7650 5400 50
+$EndSheet
+Wire Wire Line
+	7100 5400 6900 5400
+Wire Wire Line
+	7650 5400 7850 5400
+Text GLabel 7850 5400 2    50   Input ~ 0
+5V
+Text GLabel 6900 5400 0    50   Input ~ 0
+12V
+Wire Wire Line
+	2050 3900 2050 4200
+Wire Wire Line
+	2100 4200 2050 4200
+Connection ~ 2050 4200
+Wire Wire Line
+	2050 4200 2050 4750
+Wire Wire Line
+	1900 4000 1900 4100
+Wire Wire Line
+	1900 4550 1900 4650
+Wire Wire Line
+	2000 3800 2000 4500
+Wire Wire Line
+	1900 4500 2000 4500
+Connection ~ 2000 4500
+Wire Wire Line
+	2000 4500 2000 5050
+Wire Wire Line
+	1900 3800 2000 3800
+Connection ~ 2000 3800
+Wire Wire Line
+	1900 4000 2100 4000
+Wire Wire Line
+	2100 4100 2100 4000
+Wire Wire Line
+	2100 4650 2100 4550
+Wire Wire Line
+	2100 4550 1900 4550
+Wire Wire Line
+	1900 5200 1900 5150
+Wire Wire Line
+	1900 5150 2250 5150
 $EndSCHEMATC
