File: Black_STM32F407VET6/power.sch (KiCad schematic (older format))
At the start: 10 parts, among them U4 XL2012E1

Commit message: change large cap for dcdc output
Parts:
- C13: footprint Capacitor_SMD:CP_Elec_6.3x7.7 -> Capacitor_SMD:CP_Elec_8x10
Changed lines of the file:
@@
 F 0 "C13" H 7000 3750 50  0000 L CNN
 F 1 "220uF/16v" H 6750 3650 50  0000 L CNN
-F 2 "Capacitor_SMD:CP_Elec_6.3x7.7" H 7200 3700 50  0001 C CNN
+F 2 "Capacitor_SMD:CP_Elec_8x10" H 7200 3700 50  0001 C CNN
 F 3 "~" H 7200 3700 50  0001 C CNN
 	1    7200 3700
@@
 L power:GND #PWR?
 U 1 1 5D372883
-P 8300 4200
+P 8650 4300
 AR Path="/5D372883" Ref="#PWR?"  Part="1"
 AR Path="/5D345ACA/5D372883" Ref="#PWR05"  Part="1"
-F 0 "#PWR05" H 8300 3950 50  0001 C CNN
-F 1 "GND" H 8305 4027 50  0000 C CNN
-F 2 "" H 8300 4200 50  0001 C CNN
-F 3 "" H 8300 4200 50  0001 C CNN
-	1    8300 4200
+F 0 "#PWR05" H 8650 4050 50  0001 C CNN
+F 1 "GND" H 8655 4127 50  0000 C CNN
+F 2 "" H 8650 4300 50  0001 C CNN
+F 3 "" H 8650 4300 50  0001 C CNN
+	1    8650 4300
 	1    0    0    -1
 $EndComp
@@
 Text HLabel 3950 3150 0    50   Input ~ 0
 12V
-Text HLabel 8550 3150 2    50   Output ~ 0
+Text HLabel 8950 3150 2    50   Output ~ 0
 5V
 $Comp
@@
 Connection ~ 8300 3150
 Wire Wire Line
-	8300 3150 8550 3150
-Wire Wire Line
 	7950 3800 7950 4100
 Wire Wire Line
@@
 	8300 4100 7950 4100
 Connection ~ 7950 4100
+Connection ~ 8300 4100
 Wire Wire Line
-	8300 4200 8300 4100
-Connection ~ 8300 4100
+	8650 4100 8300 4100
+Wire Wire Line
+	8650 4300 8650 4100
+Wire Wire Line
+	8300 3150 8950 3150
 $EndSCHEMATC
