File: Black_STM32F407VET6/STM32F407VET6.kicad_pcb (KiCad board)
At the start: 2 copper layers, 81.3 x 99.7 mm, 103 parts, among them J1 T0, J10 Fan2, J11 Fan1, J12 X_logic, J13 Microsteps, J14 X-, J15 Y-, J16 Z-, J17 Left, J18 Y_logic, J19 X+, J2 T1, J20 Y+, J21 Z+, J22 Microsteps, J23 EXP2, J24 Z_logic, J25 Bottom, J26 Microsteps, J27 EXP1, J28 E0_logic, J29 Microsteps, J3 TB, J30 Right, J31 E1_logic, J32 Microsteps, J33 X_motor, J34 Y_motor, J35 Z_motor, J36 E0_motor, J37 E1_motor, J38 X, J39 Y, J4 TC, J40 Z, J41 E0, J42 E1, J43 Fan0, J44 COM, J45 USB, J47 I2C, J48 SPI, J49 SPI, J5 + VIN -, J50 SDIO, J51 Servo, J52 Servo, J53 PowerSelect, J54 Power, J55 PD11, J56 Power, J6 - HotBed +, J7 Heater0, J8 Heater1, J9 Fan3, Q1 Q_NMOS_GDS, Q2 Q_NMOS_GDS, Q3 Q_NMOS_GDS, Q4 Q_NMOS_GSD, Q5 Q_NMOS_GSD, Q6 Q_NMOS_GSD, Q7 Q_NMOS_GSD, U1 SN74AHC, U2 SN74AHC, U3 SN74AHC, U4 LM2596S-5, U5 AT24CS01-SSHM

Commit message: change dcdc chip
Parts:
- removed REF**: OSHW-Symbol_6.7x6mm_SilkScreen, Symbol:OSHW-Symbol_6.7x6mm_SilkScreen
- added C12: 1uF, Capacitor_SMD:C_0805_2012Metric, F.Cu at (145.3, 103.0)
- added C13: 220uF/16v, Capacitor_SMD:CP_Elec_6.3x7.7, F.Cu at (156.8, 107.2)
- added C14: 100nF, Capacitor_SMD:C_0805_2012Metric, F.Cu at (158.5, 102.6)
- added C15: 10uF, Capacitor_SMD:C_0805_2012Metric, F.Cu at (156.0, 123.1)
- added C16: 10uF, Capacitor_SMD:C_0805_2012Metric, F.Cu at (156.0, 125.2)
- C1, C2, C3, C4: footprint Capacitor_THT:CP_Radial_D5.0mm_P2.00mm -> Capacitor_Tantalum_SMD:CP_EIA-3216-10_Kemet-I
- C5: value 100uF 35V -> 47uF/50v; footprint Capacitor_THT:CP_Radial_D8.0mm_P3.50mm -> Capacitor_SMD:CP_Elec_6.3x7.7
- C6: value 220uF 35V -> 1uF; footprint Capacitor_THT:CP_Radial_D6.3mm_P2.50mm -> Capacitor_SMD:C_0805_2012Metric
- D1: value SS14 -> SS54; moved to F.Cu
- L1: value 47uH -> 47uH/3A; footprint Inductor_THT:L_Radial_D9.5mm_P5.00mm_Fastron_07HVP -> Inductor_SMD:L_7.3x7.3_H4.5
- Q1, Q2, Q3: value Q_NMOS_GDS -> IRLR8726PBF
- Q4, Q5, Q6, Q7: value Q_NMOS_GSD -> IRLML0030TRPBF
- U4: value LM2596S-5 -> XL2012E1; footprint Package_TO_SOT_SMD:TO-263-5_TabPin3 -> Package_SO:SOIC-8_3.9x4.9mm_P1.27mm
- moved C6 18.4 mm to (145.3, 107.1), turned to 270 degrees
- moved C5 16.0 mm to (140.5, 110.0), turned to 270 degrees
- moved L1 8.89 mm to (156.7, 114.7), turned to 0 degrees
- moved D1 6.07 mm to (148.1, 112.5)
- moved U4 5.61 mm to (149.2, 104.9), turned to 270 degrees
- moved R1 2.22 mm to (131.7, 89.7), turned to 180 degrees
- moved R2 2.22 mm to (139.3, 89.7), turned to 180 degrees
- moved R3 2.22 mm to (146.9, 89.7), turned to 180 degrees
- moved R4 2.22 mm to (154.6, 89.7), turned to 180 degrees
- moved C3 1.41 mm to (147.4, 91.6)
- moved C1 1.41 mm to (132.2, 91.6)
- moved C2 1.40 mm to (139.8, 91.6)
- moved C4 1.40 mm to (155.1, 91.6)
Connections:
- C6 pad 1: 5V -> 12V
- U4 pad 1: 12V -> 5V
- U4 pad 2: Net-(D1-Pad1) -> Net-(U4-Pad2)
- U4 pad 3: GND -> Net-(C12-Pad2)
- U4 pad 4: 5V -> 12V
- U4 pad 5: GND -> Net-(D1-Pad1)
Routing:
- net GND: track 756.5 -> 709.1 mm, vias 104 -> 64
- net Y-: track 67.5 -> 94.0 mm, vias 0 -> 1
- net 5V: track 268.4 -> 287.4 mm, vias 1 -> 3
- net Net-(C12-Pad2): track 0.00 -> 11.1 mm, vias 0 -> 2
- net 12V: track 304.2 -> 296.8 mm, vias 5 -> 4
- net 3V3: track 325.5 -> 330.9 mm
- net Net-(D1-Pad1): track 16.7 -> 12.2 mm
- net TC: track 45.4 -> 42.2 mm, vias 0 -> 1
- net X_En: track 69.6 -> 67.9 mm
- net HotBed: track 40.7 -> 39.1 mm
- net TB: track 39.4 -> 38.5 mm, vias 0 -> 1
- net T1: track 27.6 -> 26.8 mm, vias 0 -> 1
- net T0: track 22.4 -> 21.6 mm, vias 0 -> 1
- added copper zone on B.Cu, net 12V
- added copper zone on F.Cu, net 12V
- added copper zone on F.Cu, net Net-(D1-Pad1)
Other:
- board text removed: "https://github.com/jmz52/hardware"

Commit message: optimize for current
Parts:
- moved Q1 1.00 mm to (142.8, 118.5)
- moved U1 1.00 mm to (150.9, 118.5)
Routing:
- net GND: track 709.1 -> 701.0 mm, vias 64 -> 66
- net HotBed: track 39.1 -> 40.6 mm
- net 5V: track 287.4 -> 286.3 mm
- net Net-(Q1-Pad1): track 3.40 -> 4.40 mm
- added copper zone on F.Cu, net Net-(J6-Pad2)

Commit message: optimize tracks
Routing:
- net 5V: track 286.3 -> 287.1 mm
- net GND: vias 66 -> 69
Changed lines of the file:
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@@
     (thickness 1.6)
     (drawings 74)
-    (tracks 1255)
+    (tracks 1259)
     (zones 0)
     (modules 107)
@@
   (gr_arc (start 195.58 153.797) (end 195.58 155.067) (angle -90) (layer Edge.Cuts) (width 0.15))
   (gr_arc (start 116.84 153.797) (end 115.57 153.797) (angle -90) (layer Edge.Cuts) (width 0.15))
-  (via (at 148.717 116.228) (size 0.8) (drill 0.4) (layers F.Cu B.Cu) (net 7))
+  (via (at 150.495 107.061) (size 0.8) (drill 0.4) (layers F.Cu B.Cu) (net 7))
+  (via (at 155.702 105.41) (size 0.8) (drill 0.4) (layers F.Cu B.Cu) (net 7))
+  (via (at 154.051 105.41) (size 0.8) (drill 0.4) (layers F.Cu B.Cu) (net 7))
   (segment (start 181.93 132.99) (end 182.88 132.04) (width 1) (layer F.Cu) (net 1))
   (segment (start 181.93 135.795) (end 181.93 132.99) (width 1) (layer F.Cu) (net 1))
@@
   (segment (start 147.73 137.535) (end 148.91 136.355) (width 0.5) (layer F.Cu) (net 6))
   (segment (start 146 137.535) (end 147.73 137.535) (width 0.5) (layer F.Cu) (net 6))
+  (via (at 148.717 116.228) (size 0.8) (drill 0.4) (layers F.Cu B.Cu) (net 7))
   (via (at 150.622 122.682) (size 0.8) (drill 0.4) (layers F.Cu B.Cu) (net 7))
   (via (at 150.622 130.81) (size 0.8) (drill 0.4) (layers F.Cu B.Cu) (net 7))
@@
   (via (at 149.098 124.206) (size 0.8) (drill 0.4) (layers F.Cu B.Cu) (net 7))
   (via (at 154.051 104.013) (size 0.8) (drill 0.4) (layers F.Cu B.Cu) (net 7))
-  (via (at 155.575 109.855) (size 0.8) (drill 0.4) (layers F.Cu B.Cu) (net 7))
+  (via (at 155.702 109.855) (size 0.8) (drill 0.4) (layers F.Cu B.Cu) (net 7))
   (via (at 154.178 109.855) (size 0.8) (drill 0.4) (layers F.Cu B.Cu) (net 7))
-  (via (at 152.527 109.855) (size 0.8) (drill 0.4) (layers F.Cu B.Cu) (net 7))
-  (via (at 152.4 105.283) (size 0.8) (drill 0.4) (layers F.Cu B.Cu) (net 7))
-  (via (at 150.495 105.283) (size 0.8) (drill 0.4) (layers F.Cu B.Cu) (net 7))
+  (via (at 152.4 109.855) (size 0.8) (drill 0.4) (layers F.Cu B.Cu) (net 7))
+  (via (at 152.4 105.41) (size 0.8) (drill 0.4) (layers F.Cu B.Cu) (net 7))
+  (via (at 150.495 105.41) (size 0.8) (drill 0.4) (layers F.Cu B.Cu) (net 7))
   (via (at 132.08 103.378) (size 0.8) (drill 0.4) (layers F.Cu B.Cu) (net 7))
   (via (at 133.985 103.378) (size 0.8) (drill 0.4) (layers F.Cu B.Cu) (net 7))
@@
   (via (at 157.48 104.013) (size 0.8) (drill 0.4) (layers F.Cu B.Cu) (net 7))
   (via (at 155.702 104.013) (size 0.8) (drill 0.4) (layers F.Cu B.Cu) (net 7))
-  (via (at 152.4 103.886002) (size 0.8) (drill 0.4) (layers F.Cu B.Cu) (net 7))
+  (via (at 152.4 104.013) (size 0.8) (drill 0.4) (layers F.Cu B.Cu) (net 7))
   (segment (start 158.684874 120.750126) (end 165.095 114.34) (width 1) (layer F.Cu) (net 7))
   (segment (start 159.766 127) (end 158.684874 125.918874) (width 1) (layer F.Cu) (net 7))
@@
   (segment (start 152.4 146.05) (end 152.4 146.05) (width 0.5) (layer B.Cu) (net 10))
   (via (at 152.4 146.05) (size 0.8) (drill 0.4) (layers F.Cu B.Cu) (net 10))
-  (segment (start 162.6 101.64) (end 166.37 101.64) (width 1) (layer B.Cu) (net 10))
-  (segment (start 162.56 101.6) (end 162.6 101.64) (width 1) (layer B.Cu) (net 10))
-  (segment (start 163.79 91.48) (end 166.37 91.48) (width 1) (layer B.Cu) (net 10))
-  (segment (start 162.56 92.71) (end 163.79 91.48) (width 1) (layer B.Cu) (net 10))
+  (segment (start 162.6 101.64) (end 166.37 101.64) (width 1.27) (layer B.Cu) (net 10))
+  (segment (start 162.56 101.6) (end 162.6 101.64) (width 1.27) (layer B.Cu) (net 10))
+  (segment (start 163.79 91.48) (end 166.37 91.48) (width 1.27) (layer B.Cu) (net 10))
+  (segment (start 162.56 92.71) (end 163.79 91.48) (width 1.27) (layer B.Cu) (net 10))
   (segment (start 166.37 91.48) (end 173.99 91.48) (width 0.5) (layer B.Cu) (net 10))
   (segment (start 166.37 101.64) (end 173.99 101.64) (width 0.5) (layer B.Cu) (net 10))
@@
   (segment (start 159.4335 107.14) (end 159.4815 107.188) (width 1.27) (layer F.Cu) (net 10))
   (via (at 152.4 102.362) (size 0.8) (drill 0.4) (layers F.Cu B.Cu) (net 10))
-  (segment (start 162.56 101.6) (end 162.56 102.362) (width 1) (layer B.Cu) (net 10))
-  (segment (start 162.56 100.838) (end 162.56 92.71) (width 1) (layer B.Cu) (net 10))
-  (segment (start 162.56 101.6) (end 162.56 100.838) (width 1) (layer B.Cu) (net 10))
+  (segment (start 162.56 101.6) (end 162.56 102.362) (width 1.27) (layer B.Cu) (net 10))
+  (segment (start 162.56 100.838) (end 162.56 92.71) (width 1.27) (layer B.Cu) (net 10))
+  (segment (start 162.56 101.6) (end 162.56 100.838) (width 1.27) (layer B.Cu) (net 10))
   (segment (start 166.33 101.6) (end 166.37 101.64) (width 1.27) (layer F.Cu) (net 10))
-  (segment (start 159.4335 102.1865) (end 160.02 101.6) (width 2) (layer F.Cu) (net 10))
-  (segment (start 160.02 101.6) (end 166.33 101.6) (width 2) (layer F.Cu) (net 10))
-  (segment (start 159.4335 102.616) (end 159.4335 102.1865) (width 1.27) (layer F.Cu) (net 10))
   (segment (start 154.7645 128.0945) (end 154.94 128.27) (width 1.27) (layer F.Cu) (net 10))
   (segment (start 155.0185 123.063) (end 155.0185 125.222) (width 1.27) (layer F.Cu) (net 10))
   (segment (start 155.0185 128.1915) (end 154.94 128.27) (width 1.27) (layer F.Cu) (net 10))
   (segment (start 155.0185 125.222) (end 155.0185 128.1915) (width 1.27) (layer F.Cu) (net 10))
-  (segment (start 162.56 114.046) (end 162.56 102.362) (width 1) (layer B.Cu) (net 10))
-  (segment (start 154.94 121.666) (end 162.56 114.046) (width 1) (layer B.Cu) (net 10))
-  (segment (start 154.94 128.27) (end 154.94 121.666) (width 1) (layer B.Cu) (net 10))
-  (via (at 159.258 101.6) (size 0.8) (drill 0.4) (layers F.Cu B.Cu) (net 10))
-  (segment (start 159.4335 102.616) (end 159.4335 107.14) (width 2) (layer F.Cu) (net 10))
+  (segment (start 162.56 114.046) (end 162.56 102.362) (width 1.27) (layer B.Cu) (net 10))
+  (segment (start 154.94 121.666) (end 162.56 114.046) (width 1.27) (layer B.Cu) (net 10))
+  (segment (start 154.94 128.27) (end 154.94 121.666) (width 1.27) (layer B.Cu) (net 10))
+  (via (at 159.766 101.6) (size 0.8) (drill 0.4) (layers F.Cu B.Cu) (net 10))
   (segment (start 159.8545 114.7445) (end 159.8545 107.815) (width 2) (layer F.Cu) (net 10))
   (segment (start 157.734 86.36) (end 162.9 86.36) (width 1.27) (layer F.Cu) (net 10))
   (segment (start 121.92 86.36) (end 157.734 86.36) (width 1.27) (layer F.Cu) (net 10))
-  (segment (start 158.496 102.362) (end 159.258 101.6) (width 0.25) (layer B.Cu) (net 10))
-  (segment (start 152.4 102.362) (end 158.496 102.362) (width 0.25) (layer B.Cu) (net 10))
   (segment (start 151.195 102.362) (end 152.4 102.362) (width 0.25) (layer F.Cu) (net 10))
   (segment (start 151.13 102.427) (end 151.195 102.362) (width 0.25) (layer F.Cu) (net 10))
@@
   (segment (start 151.81 119.62) (end 152.4 120.21) (width 0.5) (layer F.Cu) (net 10))
   (segment (start 152.4 120.21) (end 152.4 120.65) (width 0.5) (layer F.Cu) (net 10))
+  (segment (start 159.4335 102.0595) (end 159.4335 107.14) (width 2) (layer F.Cu) (net 10))
+  (segment (start 159.893 101.6) (end 159.4335 102.0595) (width 2) (layer F.Cu) (net 10))
+  (segment (start 159.298 101.64) (end 159.258 101.6) (width 0.3) (layer F.Cu) (net 10))
+  (segment (start 159.004 102.362) (end 159.766 101.6) (width 0.25) (layer B.Cu) (net 10))
+  (segment (start 152.4 102.362) (end 159.004 102.362) (width 0.25) (layer B.Cu) (net 10))
+  (segment (start 159.806 101.64) (end 159.766 101.6) (width 0.3) (layer F.Cu) (net 10))
+  (segment (start 166.37 101.64) (end 159.806 101.64) (width 2) (layer F.Cu) (net 10))
   (segment (start 124.46 71.755) (end 124.46 76.2) (width 0.3) (layer B.Cu) (net 11))
   (segment (start 121.285 68.58) (end 124.46 71.755) (width 0.3) (layer B.Cu) (net 11))
@@
     (polygon
       (pts
-        (xy 144.9 134.4) (xy 144.9 131.826) (xy 148.082 131.826) (xy 150.368 129.54) (xy 151.892 129.54)
-        (xy 151.892 134.4)
+        (xy 144.9 134.62) (xy 144.9 132.08) (xy 147.828 132.08) (xy 150.368 129.54) (xy 151.892 129.54)
+        (xy 151.892 134.62)
       )
     )

Commit message: change large cap for dcdc output
Parts:
- C13: footprint Capacitor_SMD:CP_Elec_6.3x7.7 -> Capacitor_SMD:CP_Elec_8x10
- moved C14 2.03 mm to (158.5, 100.6)
- moved C13 1.12 mm to (157.3, 106.2)
- moved Q4 0.40 mm to (181.9, 136.4)
- moved Q5 0.40 mm to (174.3, 136.4)
- moved Q6 0.40 mm to (166.7, 136.4)
- moved Q7 0.40 mm to (159.1, 136.4)
Routing:
- net 12V: track 296.8 -> 291.8 mm
- net GND: track 701.0 -> 696.7 mm, vias 69 -> 77
- net 5V: track 287.1 -> 288.1 mm

Commit message: optimize tracks
Routing:
- net GND: vias 77 -> 74
Changed lines of the file:
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@@
     (thickness 1.6)
     (drawings 78)
-    (tracks 1271)
+    (tracks 1268)
     (zones 0)
     (modules 107)
@@
   (segment (start 146 137.535) (end 147.73 137.535) (width 0.5) (layer F.Cu) (net 6))
   (via (at 150.495 107.061) (size 0.8) (drill 0.4) (layers F.Cu B.Cu) (net 7))
-  (via (at 155.702 105.41) (size 0.8) (drill 0.4) (layers F.Cu B.Cu) (net 7))
-  (via (at 154.051 105.41) (size 0.8) (drill 0.4) (layers F.Cu B.Cu) (net 7))
   (via (at 148.717 116.228) (size 0.8) (drill 0.4) (layers F.Cu B.Cu) (net 7))
   (via (at 150.622 122.682) (size 0.8) (drill 0.4) (layers F.Cu B.Cu) (net 7))
@@
   (via (at 154.178 108.458) (size 0.8) (drill 0.4) (layers F.Cu B.Cu) (net 7))
   (via (at 152.4 108.458) (size 0.8) (drill 0.4) (layers F.Cu B.Cu) (net 7))
-  (via (at 152.4 105.41) (size 0.8) (drill 0.4) (layers F.Cu B.Cu) (net 7))
   (via (at 150.495 105.41) (size 0.8) (drill 0.4) (layers F.Cu B.Cu) (net 7))
   (via (at 132.08 103.378) (size 0.8) (drill 0.4) (layers F.Cu B.Cu) (net 7))
@@
   (segment (start 132.4865 88.2905) (end 132.461 88.265) (width 0.5) (layer F.Cu) (net 12))
   (segment (start 132.4865 89.662) (end 132.4865 88.2905) (width 0.5) (layer F.Cu) (net 12))
-  (segment (start 127 88.9) (end 121.92 88.9) (width 0.5) (layer F.Cu) (net 12))
-  (segment (start 132.461 88.265) (end 127.635 88.265) (width 0.5) (layer F.Cu) (net 12))
-  (segment (start 127.635 88.265) (end 127 88.9) (width 0.5) (layer F.Cu) (net 12))
+  (segment (start 125.984 88.9) (end 121.92 88.9) (width 0.5) (layer F.Cu) (net 12))
+  (segment (start 132.461 88.265) (end 126.619 88.265) (width 0.5) (layer F.Cu) (net 12))
+  (segment (start 126.619 88.265) (end 125.984 88.9) (width 0.5) (layer F.Cu) (net 12))
   (segment (start 135.89 66.04) (end 136.525 66.675) (width 0.3) (layer B.Cu) (net 13))
   (segment (start 134.62 66.04) (end 135.89 66.04) (width 0.3) (layer B.Cu) (net 13))
@@
   (segment (start 175.768 108.204) (end 175.768 100.584) (width 0.25) (layer B.Cu) (net 90))
   (segment (start 175.768 100.584) (end 174.497998 99.313998) (width 0.25) (layer B.Cu) (net 90))
-  (segment (start 124.46 116.84) (end 123.19 115.57) (width 0.3) (layer F.Cu) (net 90))
   (segment (start 174.497998 99.313998) (end 166.808685 99.313998) (width 0.25) (layer B.Cu) (net 90))
-  (segment (start 165.677315 99.313998) (end 166.243 99.313998) (width 0.3) (layer F.Cu) (net 90))
-  (segment (start 130.556002 99.313998) (end 165.677315 99.313998) (width 0.3) (layer F.Cu) (net 90))
-  (segment (start 127 102.87) (end 130.556002 99.313998) (width 0.3) (layer F.Cu) (net 90))
-  (segment (start 120.65 102.87) (end 127 102.87) (width 0.3) (layer F.Cu) (net 90))
-  (segment (start 119.38 104.14) (end 120.65 102.87) (width 0.3) (layer F.Cu) (net 90))
-  (segment (start 119.38 114.3) (end 119.38 104.14) (width 0.3) (layer F.Cu) (net 90))
   (segment (start 166.37 106.64) (end 168.696 108.966) (width 0.25) (layer B.Cu) (net 90))
-  (segment (start 120.65 115.57) (end 119.38 114.3) (width 0.3) (layer F.Cu) (net 90))
+  (segment (start 131.064002 99.313998) (end 165.677315 99.313998) (width 0.3) (layer F.Cu) (net 90))
+  (segment (start 127.508 102.87) (end 131.064002 99.313998) (width 0.3) (layer F.Cu) (net 90))
+  (segment (start 165.677315 99.313998) (end 166.243 99.313998) (width 0.3) (layer F.Cu) (net 90))
   (segment (start 123.19 115.57) (end 120.65 115.57) (width 0.3) (layer F.Cu) (net 90))
+  (segment (start 124.46 116.84) (end 123.19 115.57) (width 0.3) (layer F.Cu) (net 90))
+  (segment (start 120.65 115.57) (end 119.38 114.3) (width 0.3) (layer F.Cu) (net 90))
+  (segment (start 119.38 114.3) (end 119.38 104.14) (width 0.3) (layer F.Cu) (net 90))
+  (segment (start 119.38 104.14) (end 120.65 102.87) (width 0.3) (layer F.Cu) (net 90))
+  (segment (start 120.65 102.87) (end 127.508 102.87) (width 0.3) (layer F.Cu) (net 90))
   (segment (start 166.37 118.745) (end 166.37 116.84) (width 0.3) (layer F.Cu) (net 91))
   (segment (start 167.64 120.015) (end 166.37 118.745) (width 0.3) (layer F.Cu) (net 91))
